File: elec/layout/default/bme280.kicad_pcb (KiCad board)
At the start: 2 copper layers, 225.7 x 100.8 mm, 0 parts

Commit message: layout
Parts:
- added C1: Multilayer Ceramic Capacitors MLCC - SMD/SMT 100nF 10V 0402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, lib:C0402, F.Cu at (116.8, 67.9)
- added U1: , lib:LGA-8_BME280_BL, F.Cu at (116.8, 69.8)
Routing:
- net vcc: track 0.00 -> 6.03 mm
- net gnd: track 0.00 -> 1.65 mm
Changed lines of the file:
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@@
   )
   (net 0 "")
+  (net 1 "sck")
+  (net 2 "sdi")
+  (net 3 "vcc")
+  (net 4 "gnd")
+  (footprint "lib:LGA-8_BME280_BL" (layer "F.Cu")
+    (at 116.84 69.85)
+    (attr smd)
+    (fp_text reference "U1" (at 0 -4.98) (layer "F.SilkS")
+        (effects (font (size 1 1) (thickness 0.15)))
+    )
+    (fp_text value "" (at 0 4.98) (layer "F.Fab")
+        (effects (font (size 1 1) (thickness 0.15)))
+    )
+    (fp_text user "${REFERENCE}" (at 0 0) (layer "F.Fab")
+        (effects (font (size 1 1) (thickness 0.15)))
+    )
+    (fp_line (start 1.33 -1.33) (end -1.33 -1.33)
+      (stroke (width 0.15) (type solid)) (layer "F.SilkS"))
+    (fp_line (start 1.33 1.33) (end -1.33 1.33)
+      (stroke (width 0.15) (type solid)) (layer "F.SilkS"))
+    (fp_circle (center 0 0.89) (end 0.15 0.89)
+      (stroke (width 0.3) (type solid)) (fill none) (layer "F.SilkS"))
+    (fp_circle (center 0.51 -1.02) (end 0.61 -1.02)
+      (stroke (width 0.2) (type solid)) (fill none) (layer "F.SilkS"))
+    (fp_circle (center 0 0.89) (end 0.15 0.89)
+      (stroke (width 0.3) (type solid)) (fill none) (layer "Cmts.User"))
+    (fp_circle (center 0.51 -1.02) (end 0.61 -1.02)
+      (stroke (width 0.2) (type solid)) (fill none) (layer "Cmts.User"))
+    (fp_circle (center -1.25 1.25) (end -1.22 1.25)
+      (stroke (width 0.06) (type solid)) (fill none) (layer "F.Fab"))
+    (pad "1" smd oval (at 1.26 -0.98 90) (size 0.36 0.77) (layers "F.Cu" "F.Paste" "F.Mask")
+      (net 4 "gnd") (pintype "stereo"))
+    (pad "2" smd oval (at 1.26 -0.33 90) (size 0.36 0.77) (layers "F.Cu" "F.Paste" "F.Mask")
+      (net 3 "vcc") (pintype "stereo"))
+    (pad "3" smd oval (at 1.26 0.32 90) (size 0.36 0.77) (layers "F.Cu" "F.Paste" "F.Mask")
+      (net 2 "sdi") (pintype "stereo"))
+    (pad "4" smd oval (at 1.26 0.98 90) (size 0.36 0.77) (layers "F.Cu" "F.Paste" "F.Mask")
+      (net 1 "sck") (pintype "stereo"))
+    (pad "5" smd oval (at -1.26 0.98 90) (size 0.36 0.77) (layers "F.Cu" "F.Paste" "F.Mask")
+      (net 4 "gnd") (pintype "stereo"))
+    (pad "6" smd oval (at -1.26 0.32 90) (size 0.36 0.77) (layers "F.Cu" "F.Paste" "F.Mask")
+      (net 3 "vcc") (pintype "stereo"))
+    (pad "7" smd oval (at -1.26 -0.33 90) (size 0.36 0.77) (layers "F.Cu" "F.Paste" "F.Mask")
+      (net 4 "gnd") (pintype "stereo"))
+    (pad "8" smd oval (at -1.26 -0.98 90) (size 0.36 0.77) (layers "F.Cu" "F.Paste" "F.Mask")
+      (net 3 "vcc") (pintype "stereo"))
+    (model "/Users/narayanpowderly/Documents/atopile-workspace/the-everything-sensor/.ato/modules/bme280/elec/footprints/footprints.3dshapes/LGA-8_L2.5-W2.5-H0.9-P0.65.wrl"
+      (offset (xyz 0 -0 -0))
+      (scale (xyz 1 1 1))
+      (rotate (xyz 0 0 0))
+    )
+  )
+  (footprint "lib:C0402" (layer "F.Cu")
+    (at 116.838424 67.859214)
+    (descr "Capacitor SMD 0402 (1005 Metric), square (rectangular) end terminal, IPC_7351 nominal, (Body size source: IPC-SM-782 page 76, https://www.pcb-3d.com/wordpress/wp-content/uploads/ipc-sm-782a_amendment_1_and_2.pdf), generated with kicad-footprint-generator")
+    (tags "capacitor")
+    (attr smd)
+    (fp_text reference "C1" (at 0 -1.16) (layer "F.SilkS")
+        (effects (font (size 1 1) (thickness 0.15)))
+    )
+    (fp_text value "Multilayer Ceramic Capacitors MLCC - SMD/SMT 100nF 10V 0402 RoHS" (at 0 1.16) (layer "F.Fab")
+        (effects (font (size 1 1) (thickness 0.15)))
+    )
+    (fp_text user "${REFERENCE}" (at 0 0) (layer "F.Fab")
+        (effects (font (size 0.25 0.25) (thickness 0.04)))
+    )
+    (fp_line (start -0.107836 -0.36) (end 0.107836 -0.36)
+      (stroke (width 0.12) (type solid)) (layer "F.SilkS"))
+    (fp_line (start -0.107836 0.36) (end 0.107836 0.36)
+      (stroke (width 0.12) (type solid)) (layer "F.SilkS"))
+    (fp_line (start -0.91 -0.46) (end 0.91 -0.46)
+      (stroke (width 0.05) (type solid)) (layer "F.CrtYd"))
+    (fp_line (start -0.91 0.46) (end -0.91 -0.46)
+      (stroke (width 0.05) (type solid)) (layer "F.CrtYd"))
+    (fp_line (start 0.91 -0.46) (end 0.91 0.46)
+      (stroke (width 0.05) (type solid)) (layer "F.CrtYd"))
+    (fp_line (start 0.91 0.46) (end -0.91 0.46)
+      (stroke (width 0.05) (type solid)) (layer "F.CrtYd"))
+    (fp_line (start -0.5 -0.25) (end 0.5 -0.25)
+      (stroke (width 0.1) (type solid)) (layer "F.Fab"))
+    (fp_line (start -0.5 0.25) (end -0.5 -0.25)
+      (stroke (width 0.1) (type solid)) (layer "F.Fab"))
+    (fp_line (start 0.5 -0.25) (end 0.5 0.25)
+      (stroke (width 0.1) (type solid)) (layer "F.Fab"))
+    (fp_line (start 0.5 0.25) (end -0.5 0.25)
+      (stroke (width 0.1) (type solid)) (layer "F.Fab"))
+    (pad "1" smd roundrect (at -0.48 0) (size 0.56 0.62) (layers "F.Cu" "F.Paste" "F.Mask") (roundrect_rratio 0.25)
+      (net 3 "vcc") (pintype "stereo"))
+    (pad "2" smd roundrect (at 0.48 0) (size 0.56 0.62) (layers "F.Cu" "F.Paste" "F.Mask") (roundrect_rratio 0.25)
+      (net 4 "gnd") (pintype "stereo"))
+    (model "${KICAD6_3DMODEL_DIR}/Capacitor_SMD.3dshapes/C_0402_1005Metric.wrl"
+      (offset (xyz 0 0 0))
+      (scale (xyz 1 1 1))
+      (rotate (xyz 0 0 0))
+    )
+  )
   (gr_circle (center 225.62 81.79) (end 227.32 81.79)
     (stroke (width 0.1) (type solid)) (fill none) (layer "Edge.Cuts"))
@@
       (xy 69.100734 49.778315)
     )
-    (stroke (width 0) (type solid)) (fill none) (layer "Edge.Cuts"))
+    (stroke (width 0.1) (type solid)) (fill none) (layer "Edge.Cuts"))
   (gr_arc (start 261.62 113.79) (mid 260.448427 116.618427) (end 257.62 117.79)
     (stroke (width 0.1) (type solid)) (layer "Edge.Cuts"))
@@
     (effects (font (size 2 2) (thickness 0.1)) (justify left bottom))
   )
+  (segment (start 117.393968 69.516806) (end 116.457608 68.580446) (width 0.25) (layer "F.Cu") (net 3))
+  (segment (start 116.171248 68.866806) (end 115.679184 68.866806) (width 0.25) (layer "F.Cu") (net 3))
+  (segment (start 116.457608 67.85602) (end 116.457608 68.580446) (width 0.25) (layer "F.Cu") (net 3))
+  (segment (start 116.457608 68.580446) (end 116.171248 68.866806) (width 0.25) (layer "F.Cu") (net 3))
+  (segment (start 116.457608 70.023382) (end 116.457608 68.580446) (width 0.25) (layer "F.Cu") (net 3))
+  (segment (start 115.679184 70.166806) (end 116.314184 70.166806) (width 0.25) (layer "F.Cu") (net 3))
+  (segment (start 116.314184 70.166806) (end 116.457608 70.023382) (width 0.25) (layer "F.Cu") (net 3))
+  (segment (start 118.199184 69.516806) (end 117.393968 69.516806) (width 0.25) (layer "F.Cu") (net 3))
+  (segment (start 117.417608 67.85602) (end 117.417608 68.623258) (width 0.25) (layer "F.Cu") (net 4))
+  (segment (start 117.661156 68.866806) (end 118.199184 68.866806) (width 0.25) (layer "F.Cu") (net 4))
+  (segment (start 117.417608 68.623258) (end 117.661156 68.866806) (width 0.25) (layer "F.Cu") (net 4))
   (group "" (id 6c1ef9f7-0f34-47bb-ac1a-76df23fb396e)
     (members
